Commit message: update:new finger in urdf

File: simulasi/arm_sim/urdf/robot_arm.urdf (robot description, URDF)
Before this commit: robot Arm_fadil, 8 links, 7 joints
Links:
- removed link finger_1
- removed link finger_2
- added link finger_11, mass 0.1; collision cylinder length=0.25 radius=0.025; visual cylinder length=0.25 radius=0.025
- added link finger_12, mass 0.1; collision cylinder length=0.25 radius=0.025; visual cylinder length=0.25 radius=0.025
- added link finger_21, mass 0.1; collision cylinder length=0.25 radius=0.025; visual cylinder length=0.25 radius=0.025
- added link finger_22, mass 0.1; collision cylinder length=0.25 radius=0.025; visual cylinder length=0.25 radius=0.025
Joints:
- added joint _F1: type fixed, parent finger_11, child finger_12, origin xyz=0.05 0.3 0 rpy=0 0 0
- added joint _F2: type fixed, parent finger_21, child finger_22, origin xyz=-0.05 0.3 0 rpy=0 0 0
- joint palm_F1: child finger_1 -> finger_11
- joint palm_F2: child finger_2 -> finger_21
